File: PassPad_KiCAD/PassPad_KiCAD.kicad_pcb (KiCad board)
At the start: 2 copper layers, 73.8 x 45.2 mm, 12 parts, among them J1 Conn_01x04_Socket, SW1 RotaryEncoder_Switch, SW2 SW_Push, U1 102010428

Commit message: added some files
Routing:
- net Net-(J1-Pin_4): track 0.00 -> 77.4 mm
Changed lines of the file:
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@@
+	)
+	(segment
+		(start 111.75949 72.66775)
+		(end 111.08525 73.34199)
+		(width 0.2)
+		(layer "B.Cu")
+		(net 6)
+	)
+	(segment
+		(start 138.5135 97.810592)
+		(end 138.5135 86.509936)
+		(width 0.2)
+		(layer "B.Cu")
+		(net 6)
+	)
+	(segment
+		(start 113.62525 72.66775)
+		(end 111.75949 72.66775)
+		(width 0.2)
+		(layer "B.Cu")
+		(net 6)
+	)
+	(segment
+		(start 114.77625 73.81875)
+		(end 113.62525 72.66775)
+		(width 0.2)
+		(layer "B.Cu")
+		(net 6)
+	)
+	(segment
+		(start 111.08525 73.34199)
+		(end 111.08525 94.667242)
+		(width 0.2)
+		(layer "B.Cu")
+		(net 6)
+	)
+	(segment
+		(start 132.109592 104.2145)
+		(end 138.5135 97.810592)
+		(width 0.2)
+		(layer "B.Cu")
+		(net 6)
+	)
+	(segment
+		(start 138.5135 86.509936)
+		(end 142.969086 82.05435)
+		(width 0.2)
+		(layer "B.Cu")
+		(net 6)
+	)
+	(segment
+		(start 120.632508 104.2145)
+		(end 132.109592 104.2145)
+		(width 0.2)
+		(layer "B.Cu")
+		(net 6)
+	)
+	(segment
+		(start 111.08525 94.667242)
+		(end 120.632508 104.2145)
+		(width 0.2)
+		(layer "B.Cu")
+		(net 6)
 	)
 	(segment
