File: PassPad_KiCAD/PassPad_KiCAD.kicad_pcb (KiCad board)
At the start: 2 copper layers, 73.8 x 45.2 mm, 12 parts, among them J1 Conn_01x04_Socket, SW1 RotaryEncoder_Switch, SW2 SW_Push, U1 102010428

Commit message: fixed PCB mistakes
Parts:
- removed D1, D3: 1N4148, Diode_THT:D_DO-35_SOD27_P7.62mm_Horizontal
- moved G*** 5.32 mm to (147.6, 100.0)
Connections:
- SW1 pad S1: Net-(D3-K) -> Net-(U1-P27/A1/D1)
- SW2 pad 2: Net-(D1-K) -> Net-(U1-D7/CSB/P1/RX)
- U1 pad 2: Net-(D3-A) -> Net-(U1-P27/A1/D1)
- U1 pad 4: Net-(J1-Pin_3) -> unconnected-(U1-P29/A3/D3-Pad4)
- U1 pad 6: unconnected-(U1-P7/SCL/D5-Pad6)_1 -> Net-(J1-Pin_3)
- U1 pad 8: Net-(D1-A) -> Net-(U1-D7/CSB/P1/RX)
Routing:
- net Net-(D3-A): track 46.1 -> 0.00 mm
- net Net-(J1-Pin_4): track 77.4 -> 31.6 mm
- net GND: track 162.4 -> 122.1 mm
- net Net-(J1-Pin_3): track 73.6 -> 35.2 mm
- net Net-(U1-D7/CSB/P1/RX): track 0.00 -> 36.9 mm
- net Net-(D1-K): track 33.7 -> 0.00 mm
- net Net-(U1-P27/A1/D1): track 0.00 -> 31.9 mm
- net Net-(D3-K): track 14.6 -> 0.00 mm
- net Net-(D1-A): track 8.27 -> 0.00 mm
- net Net-(U1-P26/A0/D0): track 41.9 -> 34.6 mm
- net Net-(U1-P28/A2/D2): track 41.1 -> 34.7 mm
- net +3V3: track 52.3 -> 50.8 mm
Other:
- board text added: "PassPAD v2"
- board text removed: "PassPAD v1"
